File: 01-Electronics-CarrierC/C3-Carrier-RevC.sch (EAGLE design)
At the start: 56 parts, among them J1 18650 CELL, J2 LEFT MOTOR, J3 RIGHT MOTOR, J4 RUN SWITCH, J5 USB4125-GF-A-0190, Q1 FS8205A (Fortune TSSOP8), U1 ESP32-C3 SuperMini, U2 TC1508A, U3 TP4056-42-ESOP8, U4 DW01A-G, U5 MT3608, U6 TXU0104PWR

Commit message: Sync current Scout guide, firmware, Faces and v8 cases
Parts:
- C1: value 100uF / 25V -> 100uF / 25V (FM)
- J5: value USB4125-GF-A-0190 -> TYPE-C 6P (SHOU HAN)
- Q1: value FS8205A (Fortune TSSOP8) -> 8205A (TECH PUBLIC)
- U4: value DW01A-G -> DW01A (PUOLOP)
Changed lines of the file:
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@@
 <setting verticaltext="up"/>
 </settings>
-<grid distance="0.1" unitdist="inch" unit="inch" style="lines" multiple="1" display="no" altdistance="0.01" altunitdist="inch" altunit="inch"/>
+<grid distance="0.001" unitdist="mm" unit="mm" style="lines" multiple="1" display="no" altdistance="0.01" altunitdist="inch" altunit="inch"/>
 <layers>
 <layer number="1" name="Top" color="4" fill="1" visible="no" active="no"/>
@@
 <attribute name="FUNCTION" value="CHARGE_PROTECT"/>
 </part>
-<part name="U4" library="C3_SCOUT_REVC" deviceset="DW01A" device="" value="DW01A-G">
+<part name="U4" library="C3_SCOUT_REVC" deviceset="DW01A" device="" value="DW01A (PUOLOP)">
 <attribute name="FUNCTION" value="CHARGE_PROTECT"/>
 </part>
-<part name="Q1" library="C3_SCOUT_REVC" deviceset="FS8205A" device="" value="FS8205A (Fortune TSSOP8)">
+<part name="Q1" library="C3_SCOUT_REVC" deviceset="FS8205A" device="" value="8205A (TECH PUBLIC)">
 <attribute name="FUNCTION" value="CHARGE_PROTECT"/>
 </part>
@@
 <attribute name="FUNCTION" value="RUN_BOOST"/>
 </part>
-<part name="J5" library="C3_SCOUT_REVC" deviceset="USBC" device="" value="USB4125-GF-A-0190">
+<part name="J5" library="C3_SCOUT_REVC" deviceset="USBC" device="" value="TYPE-C 6P (SHOU HAN)">
 <attribute name="FUNCTION" value="CHARGE_PROTECT"/>
 </part>
@@
 <attribute name="FUNCTION" value="RUN_BOOST"/>
 </part>
-<part name="C1" library="C3_SCOUT_REVC" deviceset="RADIAL-6.3-2.5" device="" value="100uF / 25V">
+<part name="C1" library="C3_SCOUT_REVC" deviceset="RADIAL-6.3-2.5" device="" value="100uF / 25V (FM)">
 <attribute name="FUNCTION" value="MOTOR_INTERFACE"/>
 </part>
@@
 <instances>
 <instance part="J5" gate="G$1" x="38.1" y="165.1" smashed="yes">
-<attribute name="NAME" x="25.4" y="190.5" size="1.524" layer="95"/>
-<attribute name="VALUE" x="25.4" y="184.404" size="1.524" layer="96"/>
+<attribute name="NAME" x="25.4" y="190.5" size="1.524" layer="95" font="vector"/>
+<attribute name="VALUE" x="25.4" y="184.404" size="1.524" layer="96" font="vector"/>
 </instance>
 <instance part="R2" gate="G$1" x="76.2" y="149.86" smashed="yes" rot="R270">
@@
 </instance>
 <instance part="U4" gate="G$1" x="180.34" y="76.2" smashed="yes">
-<attribute name="NAME" x="167.64" y="99.06" size="1.524" layer="95"/>
-<attribute name="VALUE" x="167.64" y="92.964" size="1.524" layer="96"/>
+<attribute name="NAME" x="167.64" y="99.06" size="1.524" layer="95" font="vector"/>
+<attribute name="VALUE" x="167.64" y="92.964" size="1.524" layer="96" font="vector"/>
 </instance>
 <instance part="R7" gate="G$1" x="236.22" y="83.82" smashed="yes" rot="R180">
@@
 </instance>
 <instance part="Q1" gate="A" x="292.1" y="60.96" smashed="yes">
-<attribute name="NAME" x="276.86" y="43.18" size="1.524" layer="95"/>
-<attribute name="VALUE" x="276.86" y="37.084" size="1.524" layer="96"/>
+<attribute name="NAME" x="276.86" y="43.18" size="1.524" layer="95" font="vector"/>
+<attribute name="VALUE" x="276.86" y="37.084" size="1.524" layer="96" font="vector"/>
 </instance>
 <instance part="Q1" gate="B" x="355.6" y="60.96" smashed="yes">
-<attribute name="NAME" x="345.44" y="43.18" size="1.524" layer="95"/>
-<attribute name="VALUE" x="345.44" y="37.084" size="1.524" layer="96"/>
+<attribute name="NAME" x="345.44" y="43.18" size="1.524" layer="95" font="vector"/>
+<attribute name="VALUE" x="345.44" y="37.084" size="1.524" layer="96" font="vector"/>
 </instance>
 </instances>
@@
 <net name="USB5V" class="3">
 <segment>
-<pinref part="J5" gate="G$1" pin="VBUS@A9"/>
-<pinref part="J5" gate="G$1" pin="VBUS@B9"/>
 <pinref part="C3" gate="G$1" pin="1"/>
 <pinref part="U3" gate="G$1" pin="VCC"/>
@@
 <junction x="63.5" y="182.88"/>
 <label x="106.68" y="207.01" size="1.524" layer="95"/>
+<pinref part="J5" gate="G$1" pin="VBUS@A9"/>
+<pinref part="J5" gate="G$1" pin="VBUS@B9"/>
 </segment>
 </net>
 <net name="CC1" class="0">
 <segment>
-<pinref part="J5" gate="G$1" pin="CC1"/>
 <pinref part="R2" gate="G$1" pin="1"/>
 <wire x1="55.88" y1="167.64" x2="76.2" y2="167.64" width="0.1524" layer="91"/>
 <wire x1="76.2" y1="154.94" x2="76.2" y2="167.64" width="0.1524" layer="91"/>
+<pinref part="J5" gate="G$1" pin="CC1"/>
 </segment>
 </net>
 <net name="CC2" class="0">
 <segment>
-<pinref part="J5" gate="G$1" pin="CC2"/>
 <pinref part="R3" gate="G$1" pin="1"/>
 <wire x1="55.88" y1="157.48" x2="101.6" y2="157.48" width="0.1524" layer="91"/>
 <wire x1="101.6" y1="144.78" x2="101.6" y2="157.48" width="0.1524" layer="91"/>
+<pinref part="J5" gate="G$1" pin="CC2"/>
 </segment>
 </net>
@@
 </segment>
 <segment>
-<pinref part="J5" gate="G$1" pin="GND@A12"/>
-<pinref part="J5" gate="G$1" pin="GND@B12"/>
-<pinref part="J5" gate="G$1" pin="SH@1"/>
-<pinref part="J5" gate="G$1" pin="SH@2"/>
-<pinref part="J5" gate="G$1" pin="SH@3"/>
-<pinref part="J5" gate="G$1" pin="SH@4"/>
 <wire x1="27.94" y1="129.54" x2="27.94" y2="139.7" width="0.1524" layer="91"/>
 <wire x1="27.94" y1="129.54" x2="33.02" y2="129.54" width="0.1524" layer="91"/>
@@
 <junction x="33.02" y="129.54"/>
 <label x="57.912" y="127" size="1.524" layer="95"/>
+<pinref part="J5" gate="G$1" pin="GND@A12"/>
+<pinref part="J5" gate="G$1" pin="GND@B12"/>
+<pinref part="J5" gate="G$1" pin="SH@1"/>
+<pinref part="J5" gate="G$1" pin="SH@2"/>
+<pinref part="J5" gate="G$1" pin="SH@3"/>
+<pinref part="J5" gate="G$1" pin="SH@4"/>
 </segment>
 <segment>
@@
 </segment>
 <segment>
-<pinref part="Q1" gate="B" pin="S"/>
 <wire x1="360.68" y1="43.18" x2="360.68" y2="50.8" width="0.1524" layer="91"/>
 <label x="365.252" y="40.64" size="1.524" layer="95"/>
+<pinref part="Q1" gate="B" pin="S"/>
 </segment>
 <segment>
@@
 <pinref part="R6" gate="G$1" pin="2"/>
 <pinref part="C5" gate="G$1" pin="1"/>
-<pinref part="U4" gate="G$1" pin="VCC"/>
 <wire x1="106.68" y1="91.44" x2="129.54" y2="91.44" width="0.1524" layer="91"/>
 <wire x1="129.54" y1="78.74" x2="129.54" y2="91.44" width="0.1524" layer="91"/>
@@
 <wire x1="154.94" y1="83.82" x2="165.1" y2="83.82" width="0.1524" layer="91"/>
 <junction x="129.54" y="91.44"/>
+<pinref part="U4" gate="G$1" pin="VCC"/>
 </segment>
 </net>
@@
 <pinref part="J1" gate="G$1" pin="2"/>
 <pinref part="C5" gate="G$1" pin="2"/>
-<pinref part="U4" gate="G$1" pin="VSS"/>
-<pinref part="Q1" gate="A" pin="S"/>
 <wire x1="53.34" y1="68.58" x2="73.66" y2="68.58" width="0.1524" layer="91"/>
 <wire x1="73.66" y1="50.8" x2="73.66" y2="68.58" width="0.1524" layer="91"/>
@@
 <junction x="129.54" y="50.8"/>
 <label x="86.36" y="52.07" size="1.524" layer="95"/>
+<pinref part="U4" gate="G$1" pin="VSS"/>
+<pinref part="Q1" gate="A" pin="S"/>
 </segment>
 </net>
 <net name="CS" class="0">
 <segment>
-<pinref part="U4" gate="G$1" pin="CS"/>
 <pinref part="R7" gate="G$1" pin="2"/>
 <wire x1="195.58" y1="83.82" x2="231.14" y2="83.82" width="0.1524" layer="91"/>
+<pinref part="U4" gate="G$1" pin="CS"/>
 </segment>
 </net>
 <net name="OD" class="0">
 <segment>
-<pinref part="U4" gate="G$1" pin="OD"/>
-<pinref part="Q1" gate="A" pin="G"/>
 <wire x1="195.58" y1="66.04" x2="261.62" y2="66.04" width="0.1524" layer="91"/>
 <wire x1="261.62" y1="60.96" x2="261.62" y2="66.04" width="0.1524" layer="91"/>
 <wire x1="261.62" y1="60.96" x2="281.94" y2="60.96" width="0.1524" layer="91"/>
+<pinref part="U4" gate="G$1" pin="OD"/>
+<pinref part="Q1" gate="A" pin="G"/>
 </segment>
 </net>
 <net name="OC" class="0">
 <segment>
-<pinref part="U4" gate="G$1" pin="OC"/>
-<pinref part="Q1" gate="B" pin="G"/>
 <wire x1="195.58" y1="73.66" x2="256.54" y2="73.66" width="0.1524" layer="91"/>
 <wire x1="256.54" y1="73.66" x2="256.54" y2="99.06" width="0.1524" layer="91"/>
@@
 <wire x1="335.28" y1="60.96" x2="335.28" y2="99.06" width="0.1524" layer="91"/>
 <wire x1="335.28" y1="60.96" x2="345.44" y2="60.96" width="0.1524" layer="91"/>
+<pinref part="U4" gate="G$1" pin="OC"/>
+<pinref part="Q1" gate="B" pin="G"/>
 </segment>
 </net>
 <net name="D12" class="1">
 <segment>
-<pinref part="Q1" gate="A" pin="D"/>
-<pinref part="Q1" gate="B" pin="D"/>
 <wire x1="297.18" y1="71.12" x2="297.18" y2="81.28" width="0.1524" layer="91"/>
 <wire x1="297.18" y1="81.28" x2="360.68" y2="81.28" width="0.1524" layer="91"/>
 <wire x1="360.68" y1="71.12" x2="360.68" y2="81.28" width="0.1524" layer="91"/>
+<pinref part="Q1" gate="A" pin="D"/>
+<pinref part="Q1" gate="B" pin="D"/>
 </segment>
 </net>
@@
 </instance>
 <instance part="C1" gate="G$1" x="243.84" y="182.88" smashed="yes" rot="R270">
-<attribute name="NAME" x="248.92" y="195.58" size="1.524" layer="95"/>
-<attribute name="VALUE" x="248.92" y="189.484" size="1.524" layer="96"/>
+<attribute name="NAME" x="248.92" y="195.58" size="1.524" layer="95" font="vector"/>
+<attribute name="VALUE" x="248.92" y="189.484" size="1.524" layer="96" font="vector"/>
 </instance>
 </instances>
@@
 </segment>
 <segment>
-<pinref part="C1" gate="G$1" pin="2"/>
 <wire x1="243.84" y1="175.26" x2="243.84" y2="177.8" width="0.1524" layer="91"/>
 <label x="248.412" y="172.72" size="1.524" layer="95"/>
+<pinref part="C1" gate="G$1" pin="2"/>
 </segment>
 <segment>
@@
 <pinref part="U2" gate="G$1" pin="VDD@8"/>
 <pinref part="C2" gate="G$1" pin="1"/>
-<pinref part="C1" gate="G$1" pin="1"/>
 <wire x1="210.82" y1="187.96" x2="210.82" y2="208.28" width="0.1524" layer="91"/>
 <wire x1="210.82" y1="208.28" x2="243.84" y2="208.28" width="0.1524" layer="91"/>
@@
 <junction x="243.84" y="208.28"/>
 <label x="259.08" y="209.55" size="1.524" layer="95"/>
-</segment>
-<segment>
+<pinref part="C1" gate="G$1" pin="1"/>
+</segment>
+<segment>
